Commit message: xacro update

File: src/bumperbot_description/urdf/bumperbot.urdf.xacro (robot description, xacro)
@@ -13,5 +13,59 @@
     <parent link="base_footprint"/>
     <child link="base_link" />
-    <origin xyz="0 0 0.033" rpy="0 0 0"/>
+    <origin rpy="0 0 0" xyz="0 0 0.33"/>
   </joint>
+  <link name="wheel_right_link">
+    <visual>
+      <origin rpy="1.57 0 0" xyz="0 0 0"/>
+      <geometry>
+        <mesh filename="package://bumperbot_description/meshes/wheel_right_link.STL"/>
+      </geometry>
+    </visual>
+  </link>
+  <joint name="wheel_right_joint" type="continuos">
+    <parent link="base_link"/>
+    <child link="wheel_right_link"/>
+    <axis xyz="0 1 0"/>
+    <origin rpy="0 0 0" xyz="0 -0.07 0"/>
+  <joint>
+  <link name="wheel_left_link">
+    <visual>
+      <origin rpy="-1.57 0 0" xyz="0 0 0"/>
+      <geometry>
+        <mesh filename="package://bumperbot_description/meshes/wheel_left_link.STL"/>
+      </geometry>
+    </visual>
+  </link>
+  <joint name="wheel_left_joint" type="continuos">
+    <parent link="base_link"/>
+    <child link="wheel_left_link"/>
+    <axis xyz="0 1 0"/>
+    <origin rpy="0 0 0" xyz="0 0.07 0"/>
+  <joint>
+  <link name="caster_front_link">
+    <visual>
+      <origin rpy="0 0 0" xyz="0 0 0"/>
+      <geometry>
+        <mesh filename="package://bumperbot_description/meshes/caster_front_link.STL"/>
+      </geometry>
+    </visual>
+  </link>
+  <joint name="caster_front_joint" type="fixed">
+    <parent link="base_link"/>
+    <child link="caster_front_link"/>
+    <origin rpy="0 0 0" xyz="0.04755 0 -0.0275"/>
+  <joint>
+  <link name="caster_rear_link">
+    <visual>
+      <origin rpy="0 0 0" xyz="0 0 0"/>
+      <geometry>
+        <mesh filename="package://bumperbot_description/meshes/caster_rear_link.STL"/>
+      </geometry>
+    </visual>
+  </link>
+  <joint name="caster_rear_joint" type="fixed">
+    <parent link="base_link"/>
+    <child link="caster_rear_link"/>
+    <origin rpy="0 0 0" xyz="-0.04755 0 -0.0275"/>
+  <joint>
 </robot>
